File: hbridge.kicad_pcb (KiCad board)
At the start: 2 copper layers, 54 parts, among them IC1 LM5106, IC2 LM5106, P1 CONN_02X03, Q1 TPW4R50, Q10 TPW4R50, Q11 TPW4R50, Q12 TPW4R50, Q13 TPW4R50, Q14 TPW4R50, Q15 TPW4R50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

Commit message: First draft done
Parts:
- added C8: 220u, Hbridge_proto:CAP_RADIAL_13MM, F.Cu at (161.5, 55.5)
- Q1, Q10, Q11, Q12, Q13, Q14, Q15, Q16, Q17, Q18, Q19, Q2, Q20, Q3, Q4, Q5, Q6, Q7, Q8, Q9: moved to B.Cu
- moved C3 99.5 mm to (161.5, 80.5)
- moved C2 12.2 mm to (64.0, 78.0)
- moved R11 8.50 mm to (71.5, 74.5)
- moved R15 8.25 mm to (104.0, 74.5)
- moved R12 8.00 mm to (80.0, 74.5)
- moved R13 8.00 mm to (88.0, 74.5)
- moved R14 8.00 mm to (96.0, 74.5)
- moved R16 8.00 mm to (115.0, 74.5)
- moved R17 8.00 mm to (123.0, 74.5)
- moved R18 8.00 mm to (131.0, 74.5)
- moved R19 8.00 mm to (139.0, 74.5)
- moved R20 8.00 mm to (147.0, 74.5)
- moved R1 5.34 mm to (73.8, 58.0)
- moved R10 5.34 mm to (148.8, 58.0)
- moved R2 5.34 mm to (81.8, 58.0)
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Connections:
- C1 pad 2: Net-(C1-Pad2) -> GND
- C2 pad 2: Net-(C1-Pad2) -> GND
- C3 pad 2: Net-(C1-Pad2) -> GND
- C4 pad 2: Net-(C4-Pad2) -> GND
- C5 pad 2: Net-(C5-Pad2) -> GND
- IC1 pad 9: Net-(C4-Pad2) -> GND
- IC2 pad 9: Net-(C5-Pad2) -> GND
- Q1 pad 2: Net-(C1-Pad2) -> VCC
- Q10 pad 2: Net-(C1-Pad2) -> VCC
- Q2 pad 2: Net-(C1-Pad2) -> VCC
- Q3 pad 2: Net-(C1-Pad2) -> VCC
- Q4 pad 2: Net-(C1-Pad2) -> VCC
- Q5 pad 2: Net-(C1-Pad2) -> VCC
- Q6 pad 2: Net-(C1-Pad2) -> VCC
- Q7 pad 2: Net-(C1-Pad2) -> VCC
- Q8 pad 2: Net-(C1-Pad2) -> VCC
- Q9 pad 2: Net-(C1-Pad2) -> VCC
Routing:
- net (no net): track 178.7 -> 0.14 mm
- net VCC: track 0.00 -> 143.6 mm
- net GND: track 0.00 -> 134.9 mm, vias 0 -> 4
- net /M-: track 13.4 -> 58.9 mm, vias 2 -> 1
- net /M+: track 10.5 -> 47.1 mm, vias 2 -> 1
- net VDD: track 28.2 -> 57.7 mm
- net Net-(Q11-Pad1): track 0.00 -> 9.25 mm, vias 0 -> 1
- net Net-(Q20-Pad1): track 0.00 -> 9.24 mm, vias 0 -> 1
- net Net-(Q19-Pad1): track 0.00 -> 9.24 mm, vias 0 -> 1
- net Net-(Q18-Pad1): track 0.00 -> 9.24 mm, vias 0 -> 1
- net Net-(Q17-Pad1): track 0.00 -> 9.24 mm, vias 0 -> 1
- net Net-(Q16-Pad1): track 0.00 -> 9.24 mm, vias 0 -> 1
- net Net-(Q15-Pad1): track 0.00 -> 9.24 mm, vias 0 -> 1
- net Net-(Q14-Pad1): track 0.00 -> 9.24 mm, vias 0 -> 1
- net Net-(Q13-Pad1): track 0.00 -> 9.24 mm, vias 0 -> 1
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- added copper zone on B.Cu, net /M+
- added copper zone on B.Cu, net /M-
- added copper zone on B.Cu, net GND
- added copper zone on In1.Cu, net GND
- added copper zone on B.Cu, net VCC
Other:
- board outline added: 112.5 x 60 mm
- copper layers 2 -> 4
